Commit message: update

File: horiokart2021_description/urdf/robot_description.urdf (robot description, URDF)
Before this commit: robot horiokart2021_robot, 5 links, 4 joints
Links:
- link base_link: geometry visual box size=0.5 0.4 0.3
- link left_wheel_link: geometry visual cylinder length=0.05 radius=0.15
- link lrf_link: geometry visual cylinder length=0.05 radius=0.05
- link right_wheel_link: geometry visual cylinder length=0.05 radius=0.15
Joints:
- joint left_wheel_joint: axis 0 -1 0 -> 0 0 1; origin xyz=0 0.214375 0 rpy=0 0 3.14159274 -> xyz=0 0.214375 0 rpy=-1.5708 0 0
- joint right_wheel_joint: axis 0 1 0 -> 0 0 1; origin xyz=0 -0.214375 0 -> xyz=0 -0.214375 0 rpy=-1.5708 0 0

Commit message: update

File: horiokart2021_description/urdf/robot_description.urdf (robot description, URDF)
Before this commit: robot horiokart2021_robot, 5 links, 4 joints
Joints:
- joint lrf_link_joint: origin xyz=0.27 0 0.15 -> xyz=0.31 0 0.15 rpy=0 0 3.14

Commit message: add multi lidar

File: horiokart2021_description/urdf/robot_description.urdf (robot description, URDF)
Before this commit: robot horiokart2021_robot, 5 links, 4 joints
Links:
- removed link lrf_link
- added link front_lrf_link; visual cylinder length=0.05 radius=0.05
- added link top_lrf_link; visual cylinder length=0.05 radius=0.05
Joints:
- removed joint lrf_link_joint
- added joint front_lrf_link_joint: type fixed, parent base_link, child front_lrf_link, origin xyz=0.31 0 0.15 rpy=0 0 3.14
- added joint top_lrf_link_joint: type fixed, parent base_link, child top_lrf_link, origin xyz=0.31 0 0.65 rpy=0 0 0

Commit message: update from horiokart in 20220903

File: horiokart2021_description/urdf/robot_description.urdf (robot description, URDF)
Before this commit: robot horiokart2021_robot, 6 links, 5 joints
Joints:
- joint base_link_joint: origin xyz=0 0 0.20316 -> xyz=0 0 0.20316 rpy=0 0 0
- joint top_lrf_link_joint: origin xyz=0.31 0 0.65 rpy=0 0 0 -> xyz=0.31 0 0.65 rpy=0 0 3.14

Commit message: update robot description

File: horiokart2021_description/urdf/robot_description.urdf (robot description, URDF)
Before this commit: robot horiokart2021_robot, 6 links, 5 joints
Joints:
- joint top_lrf_link_joint: origin xyz=0.31 0 0.65 rpy=0 0 3.14 -> xyz=0.31 0 0.33 rpy=0 0 3.14

Commit message: update robot urdf

File: horiokart2021_description/urdf/robot_description.urdf (robot description, URDF)
Before this commit: robot horiokart2021_robot, 6 links, 5 joints
Links:
- added link gps_link; visual cylinder length=0.05 radius=0.05
- added link rs_d435_link; visual box size=0.02 0.05 0.02
- added link rs_d435i_link; visual box size=0.02 0.05 0.02
- added link top_link; visual box size=0.03 0.3 0.03
Joints:
- added joint gps_link_joint: type fixed, parent base_link, child gps_link, origin xyz=0.15 0 0.33 rpy=0 0 0
- added joint rs_d435_link_joint: type fixed, parent top_link, child rs_d435_link, origin xyz=0.01 0 -0.02 rpy=0 0.35 0
- added joint rs_d435i_link_joint: type fixed, parent top_link, child rs_d435i_link, origin xyz=0.01 0 -0.01 rpy=0 0 0
- added joint top_link_joint: type fixed, parent base_link, child top_link, origin xyz=0.31 0 0.3 rpy=0 0 0
- joint top_lrf_link_joint: origin xyz=0.31 0 0.33 rpy=0 0 3.14 -> xyz=0 0 0.03 rpy=0 0 3.14; parent base_link -> top_link
