Commit message: update urdf

File: horiokart_description/urdf/sensors.xacro (robot description, xacro)
@@ -68,11 +68,12 @@
   <xacro:macro name="realsense_d435i" params=" prefix:='' attach_to:='' rpy:='0 0 0' xyz:='0 0 0' size='0.02 0.05 0.02' ">
     <xacro:unless value="${attach_to == ''}">
-      <joint name="${prefix}rs_d435i_link_joint" type="fixed">
+      <!-- <joint name="${prefix}rs_d435i_link_joint" type="fixed"> -->
+      <joint name="${prefix}camera_link_joint" type="fixed">
         <parent link="${attach_to}"/>
-        <child link="${prefix}rs_d435i_link"/>
+        <child link="${prefix}camera_link"/>
         <origin xyz="${xyz}" rpy="${rpy}"/>
       </joint>
     </xacro:unless>
-    <link name="${prefix}rs_d435i_link">
+    <link name="${prefix}camera_link">
       <visual>
         <origin xyz="0 0 0" rpy="0 0 0"/>

Commit message: update around realsense

File: horiokart_description/urdf/sensors.xacro (robot description, xacro)
@@ -68,12 +68,14 @@
   <xacro:macro name="realsense_d435i" params=" prefix:='' attach_to:='' rpy:='0 0 0' xyz:='0 0 0' size='0.02 0.05 0.02' ">
     <xacro:unless value="${attach_to == ''}">
-      <!-- <joint name="${prefix}rs_d435i_link_joint" type="fixed"> -->
-      <joint name="${prefix}camera_link_joint" type="fixed">
+      <joint name="${prefix}rs_d435i_link_joint" type="fixed">
+      <!-- <joint name="${prefix}camera_link_joint" type="fixed"> -->
         <parent link="${attach_to}"/>
-        <child link="${prefix}camera_link"/>
+        <!-- <child link="${prefix}camera_link"/> -->
+        <child link="${prefix}rs_d435i_link"/>
         <origin xyz="${xyz}" rpy="${rpy}"/>
       </joint>
     </xacro:unless>
-    <link name="${prefix}camera_link">
+    <link name="${prefix}rs_d435i_link">
+    <!-- <link name="${prefix}camera_link"> -->
       <visual>
         <origin xyz="0 0 0" rpy="0 0 0"/>

Commit message: feat: 深度センサーのtf設定を更新
- sensors.xacro: Realsense D435iノードにセンサーを追加し、リンク名を変更
- bringup_sensors.launch.py: TFの公開設定を追加

File: horiokart_description/urdf/sensors.xacro (robot description, xacro)
@@ -67,9 +67,10 @@
   </xacro:macro>
   <xacro:macro name="realsense_d435i" params=" prefix:='' attach_to:='' rpy:='0 0 0' xyz:='0 0 0' size='0.02 0.05 0.02' ">
+    <xacro:include filename="$(find realsense2_description)/urdf/_d435.urdf.xacro" />
     <xacro:unless value="${attach_to == ''}">
       <!-- <joint name="${prefix}rs_d435i_link_joint" type="fixed"> -->
-      <joint name="${prefix}camera_link_joint" type="fixed">
+      <joint name="${prefix}camera_link_base_joint" type="fixed">
         <parent link="${attach_to}"/>
-        <child link="${prefix}camera_link"/>
+        <child link="${prefix}camera_link_base"/>
         <!-- <child link="${prefix}rs_d435i_link"/> -->
         <origin xyz="${xyz}" rpy="${rpy}"/>
@@ -77,5 +78,5 @@
     </xacro:unless>
     <!-- <link name="${prefix}rs_d435i_link"> -->
-    <link name="${prefix}camera_link">
+    <link name="${prefix}camera_link_base">
       <visual>
         <origin xyz="0 0 0" rpy="0 0 0"/>
@@ -85,4 +86,8 @@
       </visual>
     </link>
+    <xacro:sensor_d435 parent="${prefix}camera_link_base" name="camera" use_nominal_extrinsics="true" add_plug="false" use_mesh="false">
+      <!-- Provide required 'origin' block expected by the sensor_d435 macro -->
+      <origin xyz="0 0 0" rpy="0 0 0"/>
+    </xacro:sensor_d435>
   </xacro:macro>
 </robot>
