Commit message: update urdf

File: horiokart_description/urdf/horiokart_description.urdf.xacro (robot description, xacro)
@@ -9,5 +9,5 @@
   <!-- top frame for sensors -->
   <joint name="top_frame_link_joint" type="fixed">
-    <origin xyz="0.31 0 0.3" rpy="0 0 0"/>
+    <origin xyz="0.23 0 0.3" rpy="0 0 0"/>
     <parent link="base_link"/>
     <child link="top_frame_link"/>

Commit message: update urdf

File: horiokart_description/urdf/horiokart_description.urdf.xacro (robot description, xacro)
@@ -9,5 +9,5 @@
   <!-- top frame for sensors -->
   <joint name="top_frame_link_joint" type="fixed">
-    <origin xyz="0.23 0 0.3" rpy="0 0 0"/>
+    <origin xyz="0.23 0 0.450" rpy="0 0 0"/>
     <parent link="base_link"/>
     <child link="top_frame_link"/>
@@ -23,5 +23,5 @@
   <xacro:lidar_2d prefix="top_" attach_to="top_frame_link" xyz="0 0 0.03" rpy="0 0 ${pi}"/>
   <xacro:lidar_3d prefix="livox_" attach_to="top_frame_link" xyz="0 0 0.06" rpy="0 0 0"/>
-  <xacro:realsense_d435i prefix="" attach_to="top_frame_link" xyz="0.01 0 -0.01" rpy="0 0 0"/>
+  <xacro:realsense_d435i prefix="" attach_to="top_frame_link" xyz="0.020 0 -0.100" rpy="0 0 0"/>
   <xacro:realsense_d435 prefix="" attach_to="top_frame_link" xyz="0.01 0 -0.02" rpy="0 0.35 0"/>
 </robot>

Commit message: feat: Realsense D435iセンサーの設定を更新
horiokart_description.urdf.xacro:
- Realsense D435iの位置をxyz="0.020 0 -0.230"に変更

sensors.xacro:
- Realsense D435iのジョイント名をカメラ用に変更し、関連するリンクを更新

File: horiokart_description/urdf/horiokart_description.urdf.xacro (robot description, xacro)
@@ -23,5 +23,5 @@
   <xacro:lidar_2d prefix="top_" attach_to="top_frame_link" xyz="0 0 0.03" rpy="0 0 ${pi}"/>
   <xacro:lidar_3d prefix="livox_" attach_to="top_frame_link" xyz="0 0 0.06" rpy="0 0 0"/>
-  <xacro:realsense_d435i prefix="" attach_to="top_frame_link" xyz="0.020 0 -0.100" rpy="0 0 0"/>
-  <xacro:realsense_d435 prefix="" attach_to="top_frame_link" xyz="0.01 0 -0.02" rpy="0 0.35 0"/>
+  <xacro:realsense_d435i prefix="" attach_to="top_frame_link" xyz="0.020 0 -0.230" rpy="0 0.288 0"/>
+  <!-- <xacro:realsense_d435 prefix="" attach_to="top_frame_link" xyz="0.01 0 -0.02" rpy="0 0.35 0"/> -->
 </robot>

File: horiokart_description/urdf/sensors.xacro (robot description, xacro)
@@ -68,14 +68,14 @@
   <xacro:macro name="realsense_d435i" params=" prefix:='' attach_to:='' rpy:='0 0 0' xyz:='0 0 0' size='0.02 0.05 0.02' ">
     <xacro:unless value="${attach_to == ''}">
-      <joint name="${prefix}rs_d435i_link_joint" type="fixed">
-      <!-- <joint name="${prefix}camera_link_joint" type="fixed"> -->
+      <!-- <joint name="${prefix}rs_d435i_link_joint" type="fixed"> -->
+      <joint name="${prefix}camera_link_joint" type="fixed">
         <parent link="${attach_to}"/>
-        <!-- <child link="${prefix}camera_link"/> -->
-        <child link="${prefix}rs_d435i_link"/>
+        <child link="${prefix}camera_link"/>
+        <!-- <child link="${prefix}rs_d435i_link"/> -->
         <origin xyz="${xyz}" rpy="${rpy}"/>
       </joint>
     </xacro:unless>
-    <link name="${prefix}rs_d435i_link">
-    <!-- <link name="${prefix}camera_link"> -->
+    <!-- <link name="${prefix}rs_d435i_link"> -->
+    <link name="${prefix}camera_link">
       <visual>
         <origin xyz="0 0 0" rpy="0 0 0"/>

Commit message: feat: Gazeboシミュレーション環境の追加
- docker-compose.yaml: Gazeboシミュレーション用のサービスを追加し、環境変数を設定
- Dockerfile.base: Gazebo FortressとROS-GZブリッジのインストールを追加
- horiokart_description.urdf.xacro: シミュレーション用の引数を追加し、各センサーにシミュレーションオプションを追加
- robot_base.urdf.xacro: 慣性マクロを追加し、シミュレーション条件下でのGazebo設定を追加
- sensors.xacro: センサーのマクロにシミュレーションオプションを追加
- CMakeLists.txt: シミュレーションパッケージの設定を追加
- bridge.yaml: ROSとGazebo間のトピックブリッジ設定を追加
- bringup.launch.py: シミュレーション用のロボットをスポーンするためのランチャーを追加
- package.xml: シミュレーションパッケージのメタデータを追加
- warehouse.sdf: Gazeboシミュレーション用のワールドを追加

File: horiokart_description/urdf/horiokart_description.urdf.xacro (robot description, xacro)
@@ -3,8 +3,9 @@
   <xacro:include filename="$(find horiokart_description)/urdf/robot_base.urdf.xacro" />
   <xacro:include filename="$(find horiokart_description)/urdf/sensors.xacro"/>
-  <xacro:horiokart_base/>
+  <xacro:arg name="simulation" default="false"/>
+  <xacro:horiokart_base simulation="$(arg simulation)"/>
   <!-- <xacro:lidar_2d prefix="front_" attach_to="base_link" xyz="0.31 0 0.15"  rpy="0 0 0"/> -->
-  <xacro:lidar_2d prefix="front_" attach_to="base_link" xyz="0.32 0 0.15" rpy="0 0 ${pi}"/>
-  <xacro:gps prefix="" attach_to="base_link" xyz="0.26 -0.13 0.33" rpy="0 0 0"/>
+  <xacro:lidar_2d prefix="front_" attach_to="base_link" xyz="0.32 0 0.15" rpy="0 0 ${pi}" simulation="$(arg simulation)" sensor_name="front"/>
+  <xacro:gps prefix="" attach_to="base_link" xyz="0.26 -0.13 0.33" rpy="0 0 0" simulation="$(arg simulation)"/>
   <!-- top frame for sensors -->
   <joint name="top_frame_link_joint" type="fixed">
@@ -21,7 +22,7 @@
     </visual>
   </link>
-  <xacro:lidar_2d prefix="top_" attach_to="top_frame_link" xyz="0 0 0.03" rpy="0 0 ${pi}"/>
+  <xacro:lidar_2d prefix="top_" attach_to="top_frame_link" xyz="0 0 0.03" rpy="0 0 ${pi}" simulation="$(arg simulation)" sensor_name="top"/>
   <xacro:lidar_3d prefix="livox_" attach_to="top_frame_link" xyz="0 0 0.06" rpy="0 0 0"/>
   <!-- <xacro:realsense_d435i prefix="" attach_to="top_frame_link" xyz="0.020 0 -0.230" rpy="0 0.288 0"/> -->
-  <xacro:realsense_d435i prefix="" attach_to="top_frame_link" xyz="0.020 0 -0.230" rpy="0 0.27 0"/>
+  <xacro:realsense_d435i prefix="" attach_to="top_frame_link" xyz="0.020 0 -0.230" rpy="0 0.27 0" simulation="$(arg simulation)"/>
 </robot>

File: horiokart_description/urdf/robot_base.urdf.xacro (robot description, xacro)
@@ -1,8 +1,34 @@
 <?xml version="1.0" encoding="utf-8"?>
 <robot xmlns:xacro="http://ros.org/wiki/xacro" name="horiokart">
-  <xacro:macro name="horiokart_base" >
+  <xacro:macro name="box_inertia" params="m x y z">
+    <inertial>
+      <mass value="${m}"/>
+      <inertia ixx="${m*(y*y+z*z)/12}" ixy="0" ixz="0"
+               iyy="${m*(x*x+z*z)/12}" iyz="0"
+               izz="${m*(x*x+y*y)/12}"/>
+    </inertial>
+  </xacro:macro>
+  <xacro:macro name="cylinder_inertia" params="m r h">
+    <inertial>
+      <mass value="${m}"/>
+      <inertia ixx="${m*(3*r*r+h*h)/12}" ixy="0" ixz="0"
+               iyy="${m*(3*r*r+h*h)/12}" iyz="0"
+               izz="${m*r*r/2}"/>
+    </inertial>
+  </xacro:macro>
+  <xacro:macro name="sphere_inertia" params="m r">
+    <inertial>
+      <mass value="${m}"/>
+      <inertia ixx="${2*m*r*r/5}" ixy="0" ixz="0"
+               iyy="${2*m*r*r/5}" iyz="0"
+               izz="${2*m*r*r/5}"/>
+    </inertial>
+  </xacro:macro>
+  <xacro:macro name="horiokart_base" params="simulation:=false" >
     <!-- =============== Link & Joint =============== -->
     <!-- Base -->
-    <link name="base_footprint"/>
+    <link name="base_footprint">
+      <xacro:sphere_inertia m="0.001" r="0.001"/>
+    </link>
     <joint name="base_link_joint" type="fixed">
       <origin xyz="0 0 0.15" rpy="0 0 0"/>
@@ -23,4 +49,5 @@
         </geometry>
       </collision>
+      <xacro:box_inertia m="20.0" x="0.6" y="0.4" z="0.3"/>
     </link>
     <joint name="right_wheel_joint" type="continuous">
@@ -41,4 +68,5 @@
         </geometry>
       </collision>
+      <xacro:cylinder_inertia m="1.0" r="0.15" h="0.05"/>
     </link>
     <joint name="left_wheel_joint" type="continuous">
@@ -59,4 +87,5 @@
         </geometry>
       </collision>
+      <xacro:cylinder_inertia m="1.0" r="0.15" h="0.05"/>
     </link>
     <joint name="caster_joint" type="fixed">
@@ -76,5 +105,44 @@
         </geometry>
       </collision>
+      <xacro:sphere_inertia m="0.5" r="0.05"/>
     </link>
+    <xacro:if value="${simulation}">
+      <gazebo reference="base_link">
+        <preserveFixedJoint>true</preserveFixedJoint>
+      </gazebo>
+      <gazebo reference="right_wheel_link">
+        <mu1>1.0</mu1>
+        <mu2>0.5</mu2>
+        <kp>1e6</kp>
+        <kd>100.0</kd>
+      </gazebo>
+      <gazebo reference="left_wheel_link">
+        <mu1>1.0</mu1>
+        <mu2>0.5</mu2>
+        <kp>1e6</kp>
+        <kd>100.0</kd>
+      </gazebo>
+      <gazebo reference="caster_link">
+        <mu1>0.0</mu1>
+        <mu2>0.0</mu2>
+        <kp>1e6</kp>
+        <kd>100.0</kd>
+      </gazebo>
+      <gazebo>
+        <plugin filename="ignition-gazebo-diff-drive-system"
+                name="ignition::gazebo::systems::DiffDrive">
+          <left_joint>left_wheel_joint</left_joint>
+          <right_joint>right_wheel_joint</right_joint>
+          <wheel_separation>0.5</wheel_separation>
+          <wheel_radius>0.15</wheel_radius>
+          <topic>/cmd_vel</topic>
+          <odom_topic>/odom</odom_topic>
+          <tf_topic>/tf</tf_topic>
+          <frame_id>odom</frame_id>
+          <child_frame_id>base_footprint</child_frame_id>
+          <odom_publish_frequency>50</odom_publish_frequency>
+        </plugin>
+      </gazebo>
+    </xacro:if>
   </xacro:macro>
 </robot>

File: horiokart_description/urdf/sensors.xacro (robot description, xacro)
@@ -1,5 +1,5 @@
 <?xml version="1.0" encoding="utf-8"?>
 <robot xmlns:xacro="http://ros.org/wiki/xacro" name="horiokart_v2">
-  <xacro:macro name="lidar_2d" params=" prefix:='' attach_to:='' rpy:='0 0 0' xyz:='0 0 0' length='0.05' radius='0.05' ">
+  <xacro:macro name="lidar_2d" params=" prefix:='' attach_to:='' rpy:='0 0 0' xyz:='0 0 0' length='0.05' radius='0.05' simulation:=false sensor_name:='lidar' ">
     <xacro:unless value="${attach_to == ''}">
       <joint name="${prefix}lrf_link_joint" type="fixed">
@@ -16,4 +16,30 @@
       </visual>
     </link>
+    <xacro:if value="${simulation}">
+      <gazebo reference="${prefix}lrf_link">
+        <sensor name="${sensor_name}_lidar" type="gpu_lidar">
+          <update_rate>10</update_rate>
+          <topic>/${sensor_name}_lidar_scan</topic>
+          <ignition_frame_id>${prefix}lrf_link</ignition_frame_id>
+          <lidar>
+            <scan>
+              <horizontal>
+                <samples>360</samples>
+                <resolution>1</resolution>
+                <min_angle>-3.14159</min_angle>
+                <max_angle>3.14159</max_angle>
+              </horizontal>
+            </scan>
+            <range>
+              <min>0.1</min>
+              <max>30.0</max>
+              <resolution>0.01</resolution>
+            </range>
+          </lidar>
+          <alwaysOn>true</alwaysOn>
+          <visualize>true</visualize>
+        </sensor>
+      </gazebo>
+    </xacro:if>
   </xacro:macro>
   <xacro:macro name="lidar_3d" params=" prefix:='' attach_to:='' rpy:='0 0 0' xyz:='0 0 0' length='0.05' radius='0.05' ">
@@ -33,5 +59,5 @@
     </link>
   </xacro:macro>
-  <xacro:macro name="gps" params=" prefix:='' attach_to:='' rpy:='0 0 0' xyz:='0 0 0' length='0.05' radius='0.05' ">
+  <xacro:macro name="gps" params=" prefix:='' attach_to:='' rpy:='0 0 0' xyz:='0 0 0' length='0.05' radius='0.05' simulation:=false ">
     <xacro:unless value="${attach_to == ''}">
       <joint name="${prefix}gps_link_joint" type="fixed">
@@ -48,4 +74,14 @@
       </visual>
     </link>
+    <xacro:if value="${simulation}">
+      <gazebo reference="${prefix}gps_link">
+        <sensor name="navsat" type="navsat">
+          <update_rate>1</update_rate>
+          <topic>/navsat</topic>
+          <ignition_frame_id>${prefix}gps_link</ignition_frame_id>
+          <alwaysOn>true</alwaysOn>
+        </sensor>
+      </gazebo>
+    </xacro:if>
   </xacro:macro>
   <xacro:macro name="realsense_d435" params=" prefix:='' attach_to:='' rpy:='0 0 0' xyz:='0 0 0' size='0.02 0.05 0.02' ">
@@ -66,5 +102,5 @@
     </link>
   </xacro:macro>
-  <xacro:macro name="realsense_d435i" params=" prefix:='' attach_to:='' rpy:='0 0 0' xyz:='0 0 0' size='0.02 0.05 0.02' ">
+  <xacro:macro name="realsense_d435i" params=" prefix:='' attach_to:='' rpy:='0 0 0' xyz:='0 0 0' size='0.02 0.05 0.02' simulation:=false ">
     <xacro:include filename="$(find realsense2_description)/urdf/_d435.urdf.xacro" />
     <xacro:unless value="${attach_to == ''}">
@@ -86,8 +122,31 @@
       </visual>
     </link>
-    <xacro:sensor_d435 parent="${prefix}camera_link_base" name="camera" use_nominal_extrinsics="true" add_plug="false" use_mesh="false">
-      <!-- Provide required 'origin' block expected by the sensor_d435 macro -->
-      <origin xyz="0 0 0" rpy="0 0 0"/>
-    </xacro:sensor_d435>
+    <xacro:unless value="${simulation}">
+      <xacro:sensor_d435 parent="${prefix}camera_link_base" name="camera" use_nominal_extrinsics="true" add_plug="false" use_mesh="false">
+        <origin xyz="0 0 0" rpy="0 0 0"/>
+      </xacro:sensor_d435>
+    </xacro:unless>
+    <xacro:if value="${simulation}">
+      <gazebo reference="${prefix}camera_link_base">
+        <sensor name="rgbd_camera" type="rgbd_camera">
+          <update_rate>6</update_rate>
+          <topic>/rgbd_camera</topic>
+          <ignition_frame_id>${prefix}camera_link_base</ignition_frame_id>
+          <camera>
+            <horizontal_fov>1.5184</horizontal_fov>
+            <image>
+              <width>848</width>
+              <height>480</height>
+            </image>
+            <clip>
+              <near>0.1</near>
+              <far>10.0</far>
+            </clip>
+          </camera>
+          <alwaysOn>true</alwaysOn>
+          <visualize>true</visualize>
+        </sensor>
+      </gazebo>
+    </xacro:if>
   </xacro:macro>
 </robot>

Commit message: feat: Gazeboシミュレーションのセンサー設定を改善
- lidar_2dマクロにシミュレーションパラメータを追加し、センサーの更新レート、サンプル数、最小・最大範囲、範囲解像度、ノイズパラメータを設定可能にしました。
- odom_publish_frequencyを50から20に変更しました。

File: horiokart_description/urdf/horiokart_description.urdf.xacro (robot description, xacro)
@@ -6,5 +6,8 @@
   <xacro:horiokart_base simulation="$(arg simulation)"/>
   <!-- <xacro:lidar_2d prefix="front_" attach_to="base_link" xyz="0.31 0 0.15"  rpy="0 0 0"/> -->
-  <xacro:lidar_2d prefix="front_" attach_to="base_link" xyz="0.32 0 0.15" rpy="0 0 ${pi}" simulation="$(arg simulation)" sensor_name="front"/>
+  <!-- RPLiDAR A1M8: 8kHz sampling, 5.5Hz scan, 0.15-12.0m range, 360 samples/scan (1deg resolution) -->
+  <xacro:lidar_2d prefix="front_" attach_to="base_link" xyz="0.32 0 0.15" rpy="0 0 ${pi}" simulation="$(arg simulation)" sensor_name="front"
+    sim_update_rate="5.5" sim_samples="360" sim_min_range="0.15" sim_max_range="12.0" sim_range_resolution="0.01"
+    sim_noise_mean="0.0" sim_noise_stddev="0.015"/>
   <xacro:gps prefix="" attach_to="base_link" xyz="0.26 -0.13 0.33" rpy="0 0 0" simulation="$(arg simulation)"/>
   <!-- top frame for sensors -->
@@ -22,5 +25,8 @@
     </visual>
   </link>
-  <xacro:lidar_2d prefix="top_" attach_to="top_frame_link" xyz="0 0 0.03" rpy="0 0 ${pi}" simulation="$(arg simulation)" sensor_name="top"/>
+  <!-- RPLiDAR S2: 32kHz sampling, 10Hz scan, 0.05-30.0m range, 3200 samples/scan (0.1125deg resolution) -->
+  <xacro:lidar_2d prefix="top_" attach_to="top_frame_link" xyz="0 0 0.03" rpy="0 0 ${pi}" simulation="$(arg simulation)" sensor_name="top"
+    sim_update_rate="10" sim_samples="3200" sim_min_range="0.05" sim_max_range="30.0" sim_range_resolution="0.01"
+    sim_noise_mean="0.0" sim_noise_stddev="0.020"/>
   <xacro:lidar_3d prefix="livox_" attach_to="top_frame_link" xyz="0 0 0.06" rpy="0 0 0"/>
   <!-- <xacro:realsense_d435i prefix="" attach_to="top_frame_link" xyz="0.020 0 -0.230" rpy="0 0.288 0"/> -->

File: horiokart_description/urdf/robot_base.urdf.xacro (robot description, xacro)
@@ -141,5 +141,5 @@
           <frame_id>odom</frame_id>
           <child_frame_id>base_footprint</child_frame_id>
-          <odom_publish_frequency>50</odom_publish_frequency>
+          <odom_publish_frequency>20</odom_publish_frequency>
           <publish_odom_tf>false</publish_odom_tf>
         </plugin>

File: horiokart_description/urdf/sensors.xacro (robot description, xacro)
@@ -1,5 +1,5 @@
 <?xml version="1.0" encoding="utf-8"?>
 <robot xmlns:xacro="http://ros.org/wiki/xacro" name="horiokart_v2">
-  <xacro:macro name="lidar_2d" params=" prefix:='' attach_to:='' rpy:='0 0 0' xyz:='0 0 0' length='0.05' radius='0.05' simulation:=false sensor_name:='lidar' ">
+  <xacro:macro name="lidar_2d" params=" prefix:='' attach_to:='' rpy:='0 0 0' xyz:='0 0 0' length='0.05' radius='0.05' simulation:=false sensor_name:='lidar' sim_update_rate:=10 sim_samples:=360 sim_min_range:=0.1 sim_max_range:=30.0 sim_range_resolution:=0.01 sim_noise_mean:=0.0 sim_noise_stddev:=0.0 ">
     <xacro:unless value="${attach_to == ''}">
       <joint name="${prefix}lrf_link_joint" type="fixed">
@@ -19,5 +19,5 @@
       <gazebo reference="${prefix}lrf_link">
         <sensor name="${sensor_name}_lidar" type="gpu_lidar">
-          <update_rate>10</update_rate>
+          <update_rate>${sim_update_rate}</update_rate>
           <topic>/${sensor_name}_lidar_scan</topic>
           <ignition_frame_id>${prefix}lrf_link</ignition_frame_id>
@@ -25,5 +25,5 @@
             <scan>
               <horizontal>
-                <samples>360</samples>
+                <samples>${sim_samples}</samples>
                 <resolution>1</resolution>
                 <min_angle>-3.14159</min_angle>
@@ -32,8 +32,13 @@
             </scan>
             <range>
-              <min>0.1</min>
-              <max>30.0</max>
-              <resolution>0.01</resolution>
+              <min>${sim_min_range}</min>
+              <max>${sim_max_range}</max>
+              <resolution>${sim_range_resolution}</resolution>
             </range>
+            <noise>
+              <type>gaussian</type>
+              <mean>${sim_noise_mean}</mean>
+              <stddev>${sim_noise_stddev}</stddev>
+            </noise>
           </lidar>
           <alwaysOn>true</alwaysOn>
