Commit message: feat: box_inertiaマクロに位置パラメータを追加
robot_base.urdf.xacroファイルのbox_inertiaマクロにcx、cy、czの位置パラメータを追加し、origin要素を更新しました。また、box_inertiaの呼び出しに位置パラメータを渡すように変更しました。

File: horiokart_description/urdf/robot_base.urdf.xacro (robot description, xacro)
@@ -1,6 +1,7 @@
 <?xml version="1.0" encoding="utf-8"?>
 <robot xmlns:xacro="http://ros.org/wiki/xacro" name="horiokart">
-  <xacro:macro name="box_inertia" params="m x y z">
+  <xacro:macro name="box_inertia" params="m x y z cx:=0 cy:=0 cz:=0">
     <inertial>
+      <origin xyz="${cx} ${cy} ${cz}" rpy="0 0 0"/>
       <mass value="${m}"/>
       <inertia ixx="${m*(y*y+z*z)/12}" ixy="0" ixz="0"
@@ -49,5 +50,5 @@
         </geometry>
       </collision>
-      <xacro:box_inertia m="20.0" x="0.6" y="0.4" z="0.3"/>
+      <xacro:box_inertia m="20.0" x="0.6" y="0.4" z="0.3" cx="-0.2" cy="0" cz="0.1"/>
     </link>
     <joint name="right_wheel_joint" type="continuous">
