Commit message: feat: パッケージ名をhoriokartからmgに変更
- mg_navigation:
  - package.xmlのnameを`horiokart_navigation`から`mg_navigation`に変更
  - README.mdのlaunchファイルのパスを更新
  - amcl_watchdog_node.pyでのインポートパスを更新
  - waypoint_editor_node.pyでのインポートパスを更新
  - waypoints_follower.pyでのインポートパスを更新
  - costmap_for_bag_play.cppでの名前空間を`horiokart_navigation`から`mg_navigation`に変更
  - waypoint_navigator.cppでの名前空間を`horiokart_navigation`から`mg_navigation`に変更

- mg_simulation:
  - CMakeLists.txtのプロジェクト名を`horiokart_simulation`から`mg_simulation`に変更
  - bringup.launch.pyのパッケージ名を`horiokart_simulation`から`mg_simulation`に変更
  - package.xmlのnameを`horiokart_simulation`から`mg_simulation`に変更

- mg_simulator_client:
  - CMakeLists.txtのプロジェクト名を`horiokart_simulator_client`から`mg_simulator_client`に変更
  - bringup.launch.pyのパッケージ名を`horiokart_simulator_client`から`mg_simulator_client`に変更
  - package.xmlのnameを`horiokart_simulator_client`から`mg_simulator_client`に変更

- mg_slam:
  - CMakeLists.txtのプロジェクト名を`horiokart_slam`から`mg_slam`に変更
  - bringup_slam_toolbox.launch.pyのパッケージ名を`horiokart_slam`から`mg_slam`に変更
  - record_bag.launch.pyのパッケージ名を`horiokart_slam`から`mg_slam`に変更
  - package.xmlのnameを`horiokart_slam`から`mg_slam`に変更

- mg_utils:
  - CMakeLists.txtのプロジェクト名を`horiokart_utils`から`mg_utils`に変更
  - record_bag.launch.pyのインポートパスを更新
  - package.xmlのnameを`horiokart_utils`から`mg_utils`に変更

File: mg_description/urdf/mg_description.urdf.xacro (robot description, xacro)
@@ -1,8 +1,8 @@
 <?xml version="1.0" encoding="utf-8"?>
-<robot xmlns:xacro="http://ros.org/wiki/xacro" name="horiokart">
-  <xacro:include filename="$(find horiokart_description)/urdf/robot_base.urdf.xacro" />
-  <xacro:include filename="$(find horiokart_description)/urdf/sensors.xacro"/>
+<robot xmlns:xacro="http://ros.org/wiki/xacro" name="mg">
+  <xacro:include filename="$(find mg_description)/urdf/robot_base.urdf.xacro" />
+  <xacro:include filename="$(find mg_description)/urdf/sensors.xacro"/>
   <xacro:arg name="simulation" default="false"/>
-  <xacro:horiokart_base simulation="$(arg simulation)"/>
+  <xacro:mg_base simulation="$(arg simulation)"/>
   <!-- <xacro:lidar_2d prefix="front_" attach_to="base_link" xyz="0.31 0 0.15"  rpy="0 0 0"/> -->
   <!-- RPLiDAR A1M8: 8kHz sampling, 5.5Hz scan, 0.15-12.0m range, 360 samples/scan (1deg resolution) -->

File: mg_description/urdf/robot_base.urdf.xacro (robot description, xacro)
@@ -1,4 +1,4 @@
 <?xml version="1.0" encoding="utf-8"?>
-<robot xmlns:xacro="http://ros.org/wiki/xacro" name="horiokart">
+<robot xmlns:xacro="http://ros.org/wiki/xacro" name="mg">
   <xacro:macro name="box_inertia" params="m x y z cx:=0 cy:=0 cz:=0">
     <inertial>
@@ -26,5 +26,5 @@
     </inertial>
   </xacro:macro>
-  <xacro:macro name="horiokart_base" params="simulation:=false" >
+  <xacro:macro name="mg_base" params="simulation:=false" >
     <!-- =============== Link & Joint =============== -->
     <!-- Base -->

File: mg_description/urdf/sensors.xacro (robot description, xacro)
@@ -1,4 +1,4 @@
 <?xml version="1.0" encoding="utf-8"?>
-<robot xmlns:xacro="http://ros.org/wiki/xacro" name="horiokart_v2">
+<robot xmlns:xacro="http://ros.org/wiki/xacro" name="mg">
   <xacro:macro name="lidar_2d" params=" prefix:='' attach_to:='' rpy:='0 0 0' xyz:='0 0 0' length='0.05' radius='0.05' simulation:=false sensor_name:='lidar' sim_update_rate:=10 sim_samples:=360 sim_min_range:=0.1 sim_max_range:=30.0 sim_range_resolution:=0.01 sim_noise_mean:=0.0 sim_noise_stddev:=0.0 ">
     <xacro:unless value="${attach_to == ''}">

Commit message: refactor: mg_baseをrobot_baseに名称変更
mg_description.urdf.xacroファイル内のmg_baseをrobot_baseに変更しました。
robot_base.urdf.xacroファイル内のmg_baseマクロをrobot_baseに名称変更しました。

File: mg_description/urdf/mg_description.urdf.xacro (robot description, xacro)
@@ -4,5 +4,5 @@
   <xacro:include filename="$(find mg_description)/urdf/sensors.xacro"/>
   <xacro:arg name="simulation" default="false"/>
-  <xacro:mg_base simulation="$(arg simulation)"/>
+  <xacro:robot_base simulation="$(arg simulation)"/>
   <!-- <xacro:lidar_2d prefix="front_" attach_to="base_link" xyz="0.31 0 0.15"  rpy="0 0 0"/> -->
   <!-- RPLiDAR A1M8: 8kHz sampling, 5.5Hz scan, 0.15-12.0m range, 360 samples/scan (1deg resolution) -->

File: mg_description/urdf/robot_base.urdf.xacro (robot description, xacro)
@@ -26,5 +26,5 @@
     </inertial>
   </xacro:macro>
-  <xacro:macro name="mg_base" params="simulation:=false" >
+  <xacro:macro name="robot_base" params="simulation:=false" >
     <!-- =============== Link & Joint =============== -->
     <!-- Base -->
