Commit message: fix: RGBDカメラのセンサー設定を更新
- sensors.xacroにRGBDカメラのフレームとジョイントを追加
- カメラのパラメータを調整し、レンズと歪みの設定を追加
- bridge.yamlに新しいトピックマッピングを追加

Co-authored-by: Copilot <copilot@github.com>

File: mg_description/urdf/sensors.xacro (robot description, xacro)
@@ -133,22 +133,75 @@
     </xacro:unless>
     <xacro:if value="${simulation}">
+      <joint name="${prefix}camera_depth_frame_joint" type="fixed">
+        <parent link="${prefix}camera_link_base"/>
+        <child link="${prefix}camera_depth_frame"/>
+        <origin xyz="0 0 0" rpy="0 0 0"/>
+      </joint>
+      <link name="${prefix}camera_depth_frame"/>
+      <joint name="${prefix}camera_depth_optical_frame_joint" type="fixed">
+        <parent link="${prefix}camera_depth_frame"/>
+        <child link="${prefix}camera_depth_optical_frame"/>
+        <origin xyz="0 0 0" rpy="${-pi/2} 0 ${-pi/2}"/>
+      </joint>
+      <link name="${prefix}camera_depth_optical_frame"/>
+      <joint name="${prefix}camera_color_frame_joint" type="fixed">
+        <parent link="${prefix}camera_link_base"/>
+        <child link="${prefix}camera_color_frame"/>
+        <origin xyz="0 0.015 0" rpy="0 0 0"/>
+      </joint>
+      <link name="${prefix}camera_color_frame"/>
+      <joint name="${prefix}camera_color_optical_frame_joint" type="fixed">
+        <parent link="${prefix}camera_color_frame"/>
+        <child link="${prefix}camera_color_optical_frame"/>
+        <origin xyz="0 0 0" rpy="${-pi/2} 0 ${-pi/2}"/>
+      </joint>
+      <link name="${prefix}camera_color_optical_frame"/>
       <gazebo reference="${prefix}camera_link_base">
         <sensor name="rgbd_camera" type="rgbd_camera">
-          <update_rate>6</update_rate>
-          <topic>/rgbd_camera</topic>
           <ignition_frame_id>${prefix}camera_link_base</ignition_frame_id>
-          <camera>
+          <camera name="${prefix}rgbd_camera">
             <horizontal_fov>1.5184</horizontal_fov>
+            <lens>
+              <intrinsics>
+                <fx>434.0</fx>
+                <fy>434.0</fy>
+                <cx>424.0</cx>
+                <cy>240.0</cy>
+                <s>0</s>
+              </intrinsics>
+            </lens>
+            <distortion>
+              <k1>0.0</k1>
+              <k2>0.0</k2>
+              <k3>0.0</k3>
+              <p1>0.0</p1>
+              <p2>0.0</p2>
+              <center>0.5 0.5</center>
+            </distortion>
             <image>
               <width>848</width>
               <height>480</height>
+              <format>L8</format>
             </image>
             <clip>
-              <near>0.1</near>
-              <far>10.0</far>
+              <near>0.01</near>
+              <far>30</far>
             </clip>
+            <depth_camera>
+              <clip>
+                <near>0.1</near>
+                <far>10.0</far>
+              </clip>
+            </depth_camera>
+            <noise>
+              <type>gaussian</type>
+              <mean>0</mean>
+              <stddev>0.003</stddev>
+            </noise>
           </camera>
-          <always_on>true</always_on>
-          <visualize>true</visualize>
+          <always_on>1</always_on>
+          <update_rate>10</update_rate>
+          <visualize>false</visualize>
+          <topic>/rgbd_camera</topic>
         </sensor>
       </gazebo>
